Commit message: Add provisional inertia tags and load gazebo plugin in urdf.xacros

File: franka_description/robots/hand.urdf.xacro (robot description, xacro)
@@ -3,3 +3,8 @@
   <xacro:include filename="hand.xacro"/>
   <xacro:hand ns="panda"/>
+  <gazebo>
+    <plugin name="gazebo_ros_control" filename="libgazebo_ros_control.so">
+      <robotNamespace>/</robotNamespace>
+    </plugin>
+  </gazebo>
 </robot>

File: franka_description/robots/hand.xacro (robot description, xacro)
@@ -20,4 +20,10 @@
         </geometry>
       </collision>
+      <inertial>
+        <!-- ATTENTION! Needs to be defined correctly! -->
+        <origin xyz="0 0 0.02" rpy="0 0 0"/>
+        <mass value="0.3"/>
+        <inertia ixx="0.001"  ixy="0"  ixz="0" iyy="0.001" iyz="0" izz="0.001" />
+      </inertial>
     </link>
     <link name="${ns}_leftfinger">
@@ -32,4 +38,10 @@
         </geometry>
       </collision>
+      <inertial>
+        <!-- ATTENTION! Needs to be defined correctly! -->
+        <origin xyz="0 0 0.02" rpy="0 0 0"/>
+        <mass value="0.1"/>
+        <inertia ixx="0.001"  ixy="0"  ixz="0" iyy="0.001" iyz="0" izz="0.001" />
+      </inertial>
     </link>
     <link name="${ns}_rightfinger">
@@ -46,4 +58,10 @@
         </geometry>
       </collision>
+      <inertial>
+        <!-- ATTENTION! Needs to be defined correctly! -->
+        <origin xyz="0 0 0.02" rpy="0 0 0"/>
+        <mass value="0.1"/>
+        <inertia ixx="0.001"  ixy="0"  ixz="0" iyy="0.001" iyz="0" izz="0.001" />
+      </inertial>
     </link>
     <joint name="${ns}_finger_joint1" type="prismatic">

File: franka_description/robots/panda_arm.urdf.xacro (robot description, xacro)
@@ -3,3 +3,8 @@
   <xacro:include filename="$(find franka_description)/robots/panda_arm.xacro" />
   <xacro:panda_arm />
+  <gazebo>
+    <plugin name="gazebo_ros_control" filename="libgazebo_ros_control.so">
+      <robotNamespace>/</robotNamespace>
+    </plugin>
+  </gazebo>
 </robot>

File: franka_description/robots/panda_arm.xacro (robot description, xacro)
@@ -20,4 +20,10 @@
         </geometry>
       </collision>
+      <inertial>
+        <!-- ATTENTION! Copied from another robot! Needs to be defined correctly! -->
+        <origin xyz="-0.1 0 0.07" rpy="0 0 0"/>
+        <mass value="5"/>
+        <inertia ixx="0.05"  ixy="0"  ixz="0" iyy="0.06" iyz="0" izz="0.03" />
+      </inertial>
     </link>
     <link name="${arm_id}_link1">
@@ -32,4 +38,10 @@
         </geometry>
       </collision>
+      <inertial>
+        <!-- ATTENTION! Copied from another robot! Needs to be defined correctly! -->
+        <origin xyz="0 -0.03 0.12" rpy="0 0 0"/>
+        <mass value="4"/>
+        <inertia ixx="0.1"  ixy="0"  ixz="0" iyy="0.09" iyz="0" izz="0.02" />
+      </inertial>
     </link>
     <joint name="${arm_id}_joint1" type="revolute">
@@ -52,4 +64,10 @@
         </geometry>
       </collision>
+      <inertial>
+        <!-- ATTENTION! Copied from another robot! Needs to be defined correctly! -->
+        <origin xyz="0.0003 0.059 0.042" rpy="0 0 0"/>
+        <mass value="4"/>
+        <inertia ixx="0.05"  ixy="0"  ixz="0" iyy="0.018" iyz="0" izz="0.044" />
+      </inertial>
     </link>
     <joint name="${arm_id}_joint2" type="revolute">
@@ -72,4 +90,10 @@
         </geometry>
       </collision>
+      <inertial>
+        <!-- ATTENTION! Copied from another robot! Needs to be defined correctly! -->
+        <origin xyz="0 0.03 0.13" rpy="0 0 0"/>
+        <mass value="3"/>
+        <inertia ixx="0.08"  ixy="0"  ixz="0" iyy="0.075" iyz="0" izz="0.01" />
+      </inertial>
     </link>
     <joint name="${arm_id}_joint3" type="revolute">
@@ -92,4 +116,10 @@
         </geometry>
       </collision>
+      <inertial>
+        <!-- ATTENTION! Copied from another robot! Needs to be defined correctly! -->
+        <origin xyz="0 0.067 0.034" rpy="0 0 0"/>
+        <mass value="2.7"/>
+        <inertia ixx="0.03"  ixy="0"  ixz="0" iyy="0.01" iyz="0" izz="0.029" />
+      </inertial>
     </link>
     <joint name="${arm_id}_joint4" type="revolute">
@@ -112,4 +142,10 @@
         </geometry>
       </collision>
+      <inertial>
+        <!-- ATTENTION! Copied from another robot! Needs to be defined correctly! -->
+        <origin xyz="0.0001 0.021 0.076" rpy="0 0 0"/>
+        <mass value="1.7"/>
+        <inertia ixx="0.02"  ixy="0"  ixz="0" iyy="0.018" iyz="0" izz="0.005" />
+      </inertial>
     </link>
     <joint name="${arm_id}_joint5" type="revolute">
@@ -132,4 +168,10 @@
         </geometry>
       </collision>
+      <inertial>
+        <!-- ATTENTION! Copied from another robot! Needs to be defined correctly! -->
+        <origin xyz="0 0.0006 0.0004" rpy="0 0 0"/>
+        <mass value="1.8"/>
+        <inertia ixx="0.005"  ixy="0"  ixz="0" iyy="0.0036" iyz="0" izz="0.0047" />
+      </inertial>
     </link>
     <joint name="${arm_id}_joint6" type="revolute">
@@ -152,4 +194,10 @@
         </geometry>
       </collision>
+      <inertial>
+        <!-- ATTENTION! Copied from another robot! Needs to be defined correctly! -->
+        <origin xyz="0 0 0.02" rpy="0 0 0"/>
+        <mass value="0.3"/>
+        <inertia ixx="0.001"  ixy="0"  ixz="0" iyy="0.001" iyz="0" izz="0.001" />
+      </inertial>
     </link>
     <joint name="${arm_id}_joint7" type="revolute">

File: franka_description/robots/panda_arm_hand.urdf.xacro (robot description, xacro)
@@ -5,3 +5,8 @@
   <xacro:panda_arm />
   <xacro:hand ns="panda" rpy="0 0 ${-pi/4}" connected_to="panda_link8"/>
+  <gazebo>
+    <plugin name="gazebo_ros_control" filename="libgazebo_ros_control.so">
+      <robotNamespace>/</robotNamespace>
+    </plugin>
+  </gazebo>
 </robot>

Commit message: Add joints.yaml, so that sim works with gazebo9. Still not showing the stl in gazebo, though.

File: franka_description/robots/hand.urdf.xacro (robot description, xacro)
@@ -1,4 +1,5 @@
 <?xml version="1.0" encoding="utf-8"?>
 <robot xmlns:xacro="http://www.ros.org/wiki/xacro" name="hand">
+  <link name="world"/>
   <xacro:include filename="hand.xacro"/>
   <xacro:hand ns="panda"/>

File: franka_description/robots/panda_arm.urdf.xacro (robot description, xacro)
@@ -2,9 +2,13 @@
 <robot xmlns:xacro="http://www.ros.org/wiki/xacro" name="panda">
   <xacro:include filename="$(find franka_description)/robots/panda_arm.xacro" />
-  <xacro:panda_arm />
+  <link name="world"/>
+  <xacro:panda_arm connected_to="world"/>
   <gazebo>
     <plugin name="gazebo_ros_control" filename="libgazebo_ros_control.so">
       <robotNamespace>/</robotNamespace>
     </plugin>
+    <plugin name="gravity_compensation" filename="libGravityCompensationPlugin.so">
+      <uri>model://robot</uri>
+    </plugin>
   </gazebo>
 </robot>

File: franka_description/robots/panda_arm.xacro (robot description, xacro)
@@ -22,9 +22,17 @@
       <inertial>
         <!-- ATTENTION! Copied from another robot! Needs to be defined correctly! -->
-        <origin xyz="-0.1 0 0.07" rpy="0 0 0"/>
-        <mass value="5"/>
-        <inertia ixx="0.05"  ixy="0"  ixz="0" iyy="0.06" iyz="0" izz="0.03" />
-      </inertial>
-    </link>
+        <mass value="1.2" />
+        <origin rpy="0 0 0" xyz="0 0 0.055" />
+        <inertia ixx="0.00229" ixy="0" ixz="0" iyy="0.00216" iyz="0" izz="0.00229" />
+      </inertial>
+    </link>
+    <gazebo reference="${arm_id}_link0">
+      <kp>1000000.0</kp>
+      <kd>1.0</kd>
+      <mu1>0.8</mu1>
+      <mu2>0.8</mu2>
+      <maxVel>0.0</maxVel>
+      <minDepth>0.001</minDepth>
+    </gazebo>
     <link name="${arm_id}_link1">
       <visual>
@@ -40,9 +48,17 @@
       <inertial>
         <!-- ATTENTION! Copied from another robot! Needs to be defined correctly! -->
-        <origin xyz="0 -0.03 0.12" rpy="0 0 0"/>
-        <mass value="4"/>
-        <inertia ixx="0.1"  ixy="0"  ixz="0" iyy="0.09" iyz="0" izz="0.02" />
-      </inertial>
-    </link>
+        <mass value="2.0" />
+        <origin rpy="0 0 0" xyz="0 0 0.130" />
+        <inertia ixx="0.0136666666667" ixy="0" ixz="0" iyy="0.0118666666667" iyz="0" izz="0.003" />
+      </inertial>
+    </link>
+    <gazebo reference="${arm_id}_link1">
+      <kp>1000000.0</kp>
+      <kd>1.0</kd>
+      <mu1>0.8</mu1>
+      <mu2>0.8</mu2>
+      <maxVel>0.0</maxVel>
+      <minDepth>0.001</minDepth>
+    </gazebo>
     <joint name="${arm_id}_joint1" type="revolute">
       <safety_controller k_position="100.0" k_velocity="40.0" soft_lower_limit="-2.8973" soft_upper_limit="2.8973"/>
@@ -52,4 +68,5 @@
       <axis xyz="0 0 1"/>
       <limit effort="87" lower="-2.8973" upper="2.8973" velocity="2.1750"/>
+      <dynamics damping="0.5" friction="1.0"/>
     </joint>
     <transmission name="${arm_id}_transmission1">
@@ -57,8 +74,8 @@
       <type>transmission_interface/SimpleTransmission</type>
       <joint name="${arm_id}_joint1">
-	    <hardwareInterface>PositionJointInterface</hardwareInterface>
+	    <hardwareInterface>hardware_interface/PositionJointInterface</hardwareInterface>
       </joint>
       <actuator name="${arm_id}_motor1">
-	    <hardwareInterface>PositionJointInterface</hardwareInterface>
+	    <hardwareInterface>hardware_interface/PositionJointInterface</hardwareInterface>
 	    <mechanicalReduction>1</mechanicalReduction>
       </actuator>
@@ -77,9 +94,17 @@
       <inertial>
         <!-- ATTENTION! Copied from another robot! Needs to be defined correctly! -->
-        <origin xyz="0.0003 0.059 0.042" rpy="0 0 0"/>
-        <mass value="4"/>
-        <inertia ixx="0.05"  ixy="0"  ixz="0" iyy="0.018" iyz="0" izz="0.044" />
-      </inertial>
-    </link>
+        <mass value="2.0" />
+        <origin rpy="0 0 0" xyz="0 -0.06 0.07" />
+        <inertia ixx="0.0136666666667" ixy="0" ixz="0" iyy="0.0118666666667" iyz="0" izz="0.003" />
+      </inertial>
+    </link>
+    <gazebo reference="${arm_id}_link2">
+      <kp>1000000.0</kp>
+      <kd>1.0</kd>
+      <mu1>0.8</mu1>
+      <mu2>0.8</mu2>
+      <maxVel>0.0</maxVel>
+      <minDepth>0.001</minDepth>
+    </gazebo>
     <joint name="${arm_id}_joint2" type="revolute">
       <safety_controller k_position="100.0" k_velocity="40.0" soft_lower_limit="-1.7628" soft_upper_limit="1.7628"/>
@@ -89,4 +114,5 @@
       <axis xyz="0 0 1"/>
       <limit effort="87" lower="-1.7628" upper="1.7628" velocity="2.1750"/>
+      <dynamics damping="0.5" friction="1.0"/>
     </joint>
     <transmission name="${arm_id}_transmission2">
@@ -94,8 +120,8 @@
       <type>transmission_interface/SimpleTransmission</type>
       <joint name="${arm_id}_joint2">
-	    <hardwareInterface>PositionJointInterface</hardwareInterface>
+	    <hardwareInterface>hardware_interface/PositionJointInterface</hardwareInterface>
       </joint>
       <actuator name="${arm_id}_motor2">
-	    <hardwareInterface>PositionJointInterface</hardwareInterface>
+	    <hardwareInterface>hardware_interface/PositionJointInterface</hardwareInterface>
 	    <mechanicalReduction>1</mechanicalReduction>
       </actuator>
@@ -114,9 +140,17 @@
       <inertial>
         <!-- ATTENTION! Copied from another robot! Needs to be defined correctly! -->
-        <origin xyz="0 0.03 0.13" rpy="0 0 0"/>
-        <mass value="3"/>
-        <inertia ixx="0.08"  ixy="0"  ixz="0" iyy="0.075" iyz="0" izz="0.01" />
-      </inertial>
-    </link>
+        <mass value="2.0" />
+        <origin rpy="0 0 0" xyz="0 -0.06 0.130" />
+        <inertia ixx="0.0136666666667" ixy="0" ixz="0" iyy="0.0118666666667" iyz="0" izz="0.003" />
+      </inertial>
+    </link>
+    <gazebo reference="${arm_id}_link3">
+      <kp>1000000.0</kp>
+      <kd>1.0</kd>
+      <mu1>0.8</mu1>
+      <mu2>0.8</mu2>
+      <maxVel>0.0</maxVel>
+      <minDepth>0.001</minDepth>
+    </gazebo>
     <joint name="${arm_id}_joint3" type="revolute">
       <safety_controller k_position="100.0" k_velocity="40.0" soft_lower_limit="-2.8973" soft_upper_limit="2.8973"/>
@@ -126,4 +160,5 @@
       <axis xyz="0 0 1"/>
       <limit effort="87" lower="-2.8973" upper="2.8973" velocity="2.1750"/>
+      <dynamics damping="0.5" friction="1.0"/>
     </joint>
     <transmission name="${arm_id}_transmission3">
@@ -131,8 +166,8 @@
       <type>transmission_interface/SimpleTransmission</type>
       <joint name="${arm_id}_joint3">
-	    <hardwareInterface>PositionJointInterface</hardwareInterface>
+	    <hardwareInterface>hardware_interface/PositionJointInterface</hardwareInterface>
       </joint>
       <actuator name="${arm_id}_motor3">
-	    <hardwareInterface>PositionJointInterface</hardwareInterface>
+	    <hardwareInterface>hardware_interface/PositionJointInterface</hardwareInterface>
 	    <mechanicalReduction>1</mechanicalReduction>
       </actuator>
@@ -151,9 +186,17 @@
       <inertial>
         <!-- ATTENTION! Copied from another robot! Needs to be defined correctly! -->
-        <origin xyz="0 0.067 0.034" rpy="0 0 0"/>
-        <mass value="2.7"/>
-        <inertia ixx="0.03"  ixy="0"  ixz="0" iyy="0.01" iyz="0" izz="0.029" />
-      </inertial>
-    </link>
+        <mass value="2.0" />
+        <origin rpy="0 0 0" xyz="0 0.06 0.07" />
+        <inertia ixx="0.0136666666667" ixy="0" ixz="0" iyy="0.0118666666667" iyz="0" izz="0.003" />
+      </inertial>
+    </link>
+    <gazebo reference="${arm_id}_link4">
+      <kp>1000000.0</kp>
+      <kd>1.0</kd>
+      <mu1>0.8</mu1>
+      <mu2>0.8</mu2>
+      <maxVel>0.0</maxVel>
+      <minDepth>0.001</minDepth>
+    </gazebo>
     <joint name="${arm_id}_joint4" type="revolute">
       <safety_controller k_position="100.0" k_velocity="40.0" soft_lower_limit="-3.0718" soft_upper_limit="-0.0698"/>
@@ -163,4 +206,5 @@
       <axis xyz="0 0 1"/>
       <limit effort="87" lower="-3.0718" upper="-0.0698" velocity="2.1750"/>
+      <dynamics damping="0.5" friction="1.0"/>
     </joint>
     <transmission name="${arm_id}_transmission4">
@@ -168,8 +212,8 @@
       <type>transmission_interface/SimpleTransmission</type>
       <joint name="${arm_id}_joint4">
-	    <hardwareInterface>PositionJointInterface</hardwareInterface>
+	    <hardwareInterface>hardware_interface/PositionJointInterface</hardwareInterface>
       </joint>
       <actuator name="${arm_id}_motor4">
-	    <hardwareInterface>PositionJointInterface</hardwareInterface>
+	    <hardwareInterface>hardware_interface/PositionJointInterface</hardwareInterface>
 	    <mechanicalReduction>1</mechanicalReduction>
       </actuator>
@@ -188,9 +232,17 @@
       <inertial>
         <!-- ATTENTION! Copied from another robot! Needs to be defined correctly! -->
-        <origin xyz="0.0001 0.021 0.076" rpy="0 0 0"/>
-        <mass value="1.7"/>
-        <inertia ixx="0.02"  ixy="0"  ixz="0" iyy="0.018" iyz="0" izz="0.005" />
-      </inertial>
-    </link>
+        <mass value="2.0" />
+        <origin rpy="0 0 0" xyz="0 0 0.124" />
+        <inertia ixx="0.0126506666667" ixy="0" ixz="0" iyy="0.0108506666667" iyz="0" izz="0.003" />
+      </inertial>
+    </link>
+    <gazebo reference="${arm_id}_link5">
+      <kp>1000000.0</kp>
+      <kd>1.0</kd>
+      <mu1>0.8</mu1>
+      <mu2>0.8</mu2>
+      <maxVel>0.0</maxVel>
+      <minDepth>0.001</minDepth>
+    </gazebo>
     <joint name="${arm_id}_joint5" type="revolute">
       <safety_controller k_position="100.0" k_velocity="40.0" soft_lower_limit="-2.8973" soft_upper_limit="2.8973"/>
@@ -200,4 +252,5 @@
       <axis xyz="0 0 1"/>
       <limit effort="12" lower="-2.8973" upper="2.8973" velocity="2.6100"/>
+      <dynamics damping="0.5" friction="1.0"/>
     </joint>
     <transmission name="${arm_id}_transmission5">
@@ -205,8 +258,8 @@
       <type>transmission_interface/SimpleTransmission</type>
       <joint name="${arm_id}_joint5">
-	    <hardwareInterface>PositionJointInterface</hardwareInterface>
+	    <hardwareInterface>hardware_interface/PositionJointInterface</hardwareInterface>
       </joint>
       <actuator name="${arm_id}_motor5">
-	    <hardwareInterface>PositionJointInterface</hardwareInterface>
+	    <hardwareInterface>hardware_interface/PositionJointInterface</hardwareInterface>
 	    <mechanicalReduction>1</mechanicalReduction>
       </actuator>
@@ -225,9 +278,17 @@
       <inertial>
         <!-- ATTENTION! Copied from another robot! Needs to be defined correctly! -->
-        <origin xyz="0 0.0006 0.0004" rpy="0 0 0"/>
-        <mass value="1.8"/>
-        <inertia ixx="0.005"  ixy="0"  ixz="0" iyy="0.0036" iyz="0" izz="0.0047" />
-      </inertial>
-    </link>
+        <mass value="1.0" />
+        <origin rpy="0 0 0" xyz="0 0 0.0" />
+        <inertia ixx="0.00260416666667" ixy="0" ixz="0" iyy="0.00260416666667" iyz="0" izz="0.00260416666667" />
+      </inertial>
+    </link>
+    <gazebo reference="${arm_id}_link6">
+      <kp>1000000.0</kp>
+      <kd>1.0</kd>
+      <mu1>0.8</mu1>
+      <mu2>0.8</mu2>
+      <maxVel>0.0</maxVel>
+      <minDepth>0.001</minDepth>
+    </gazebo>
     <joint name="${arm_id}_joint6" type="revolute">
       <safety_controller k_position="100.0" k_velocity="40.0" soft_lower_limit="-0.0175" soft_upper_limit="3.7525"/>
@@ -237,4 +298,5 @@
       <axis xyz="0 0 1"/>
       <limit effort="12" lower="-0.0175" upper="3.7525" velocity="2.6100"/>
+      <dynamics damping="0.5" friction="1.0"/>
     </joint>
     <transmission name="${arm_id}_transmission6">
@@ -242,8 +304,8 @@
       <type>transmission_interface/SimpleTransmission</type>
       <joint name="${arm_id}_joint6">
-	    <hardwareInterface>PositionJointInterface</hardwareInterface>
+	    <hardwareInterface>hardware_interface/PositionJointInterface</hardwareInterface>
       </joint>
       <actuator name="${arm_id}_motor6">
-	    <hardwareInterface>PositionJointInterface</hardwareInterface>
+	    <hardwareInterface>hardware_interface/PositionJointInterface</hardwareInterface>
 	    <mechanicalReduction>1</mechanicalReduction>
       </actuator>
@@ -262,9 +324,17 @@
       <inertial>
         <!-- ATTENTION! Copied from another robot! Needs to be defined correctly! -->
-        <origin xyz="0 0 0.02" rpy="0 0 0"/>
-        <mass value="0.3"/>
-        <inertia ixx="0.001"  ixy="0"  ixz="0" iyy="0.001" iyz="0" izz="0.001" />
-      </inertial>
-    </link>
+        <mass value="0.2" />
+        <origin xyz="0 0 0" />
+        <inertia ixx="6.66666666667e-05" ixy="0" ixz="0" iyy="6.66666666667e-05" iyz="0" izz="0.00012" />
+      </inertial>
+    </link>
+    <gazebo reference="${arm_id}_link7">
+      <kp>1000000.0</kp>
+      <kd>1.0</kd>
+      <mu1>0.8</mu1>
+      <mu2>0.8</mu2>
+      <maxVel>0.0</maxVel>
+      <minDepth>0.001</minDepth>
+    </gazebo>
     <joint name="${arm_id}_joint7" type="revolute">
       <safety_controller k_position="100.0" k_velocity="40.0" soft_lower_limit="-2.8973" soft_upper_limit="2.8973"/>
@@ -274,4 +344,5 @@
       <axis xyz="0 0 1"/>
       <limit effort="12" lower="-2.8973" upper="2.8973" velocity="2.6100"/>
+      <dynamics damping="0.5" friction="1.0"/>
     </joint>
     <transmission name="${arm_id}_transmission7">
@@ -279,8 +350,8 @@
       <type>transmission_interface/SimpleTransmission</type>
       <joint name="${arm_id}_joint7">
-	    <hardwareInterface>PositionJointInterface</hardwareInterface>
+	    <hardwareInterface>hardware_interface/PositionJointInterface</hardwareInterface>
       </joint>
       <actuator name="${arm_id}_motor7">
-	    <hardwareInterface>PositionJointInterface</hardwareInterface>
+	    <hardwareInterface>hardware_interface/PositionJointInterface</hardwareInterface>
 	    <mechanicalReduction>1</mechanicalReduction>
       </actuator>
