Commit message: Add transmission tags for the arm.

File: franka_description/robots/panda_arm.xacro (robot description, xacro)
@@ -53,4 +53,15 @@
       <limit effort="87" lower="-2.8973" upper="2.8973" velocity="2.1750"/>
     </joint>
+    <transmission name="${arm_id}_transmission1">
+      <robotNamespace>/</robotNamespace>
+      <type>transmission_interface/SimpleTransmission</type>
+      <joint name="${arm_id}_joint1">
+	    <hardwareInterface>PositionJointInterface</hardwareInterface>
+      </joint>
+      <actuator name="${arm_id}_motor1">
+	    <hardwareInterface>PositionJointInterface</hardwareInterface>
+	    <mechanicalReduction>1</mechanicalReduction>
+      </actuator>
+    </transmission>
     <link name="${arm_id}_link2">
       <visual>
@@ -79,4 +90,15 @@
       <limit effort="87" lower="-1.7628" upper="1.7628" velocity="2.1750"/>
     </joint>
+    <transmission name="${arm_id}_transmission2">
+      <robotNamespace>/</robotNamespace>
+      <type>transmission_interface/SimpleTransmission</type>
+      <joint name="${arm_id}_joint2">
+	    <hardwareInterface>PositionJointInterface</hardwareInterface>
+      </joint>
+      <actuator name="${arm_id}_motor2">
+	    <hardwareInterface>PositionJointInterface</hardwareInterface>
+	    <mechanicalReduction>1</mechanicalReduction>
+      </actuator>
+    </transmission>
     <link name="${arm_id}_link3">
       <visual>
@@ -105,4 +127,15 @@
       <limit effort="87" lower="-2.8973" upper="2.8973" velocity="2.1750"/>
     </joint>
+    <transmission name="${arm_id}_transmission3">
+      <robotNamespace>/</robotNamespace>
+      <type>transmission_interface/SimpleTransmission</type>
+      <joint name="${arm_id}_joint3">
+	    <hardwareInterface>PositionJointInterface</hardwareInterface>
+      </joint>
+      <actuator name="${arm_id}_motor3">
+	    <hardwareInterface>PositionJointInterface</hardwareInterface>
+	    <mechanicalReduction>1</mechanicalReduction>
+      </actuator>
+    </transmission>
     <link name="${arm_id}_link4">
       <visual>
@@ -131,4 +164,15 @@
       <limit effort="87" lower="-3.0718" upper="-0.0698" velocity="2.1750"/>
     </joint>
+    <transmission name="${arm_id}_transmission4">
+      <robotNamespace>/</robotNamespace>
+      <type>transmission_interface/SimpleTransmission</type>
+      <joint name="${arm_id}_joint4">
+	    <hardwareInterface>PositionJointInterface</hardwareInterface>
+      </joint>
+      <actuator name="${arm_id}_motor4">
+	    <hardwareInterface>PositionJointInterface</hardwareInterface>
+	    <mechanicalReduction>1</mechanicalReduction>
+      </actuator>
+    </transmission>
     <link name="${arm_id}_link5">
       <visual>
@@ -157,4 +201,15 @@
       <limit effort="12" lower="-2.8973" upper="2.8973" velocity="2.6100"/>
     </joint>
+    <transmission name="${arm_id}_transmission5">
+      <robotNamespace>/</robotNamespace>
+      <type>transmission_interface/SimpleTransmission</type>
+      <joint name="${arm_id}_joint5">
+	    <hardwareInterface>PositionJointInterface</hardwareInterface>
+      </joint>
+      <actuator name="${arm_id}_motor5">
+	    <hardwareInterface>PositionJointInterface</hardwareInterface>
+	    <mechanicalReduction>1</mechanicalReduction>
+      </actuator>
+    </transmission>
     <link name="${arm_id}_link6">
       <visual>
@@ -183,4 +238,15 @@
       <limit effort="12" lower="-0.0175" upper="3.7525" velocity="2.6100"/>
     </joint>
+    <transmission name="${arm_id}_transmission6">
+      <robotNamespace>/</robotNamespace>
+      <type>transmission_interface/SimpleTransmission</type>
+      <joint name="${arm_id}_joint6">
+	    <hardwareInterface>PositionJointInterface</hardwareInterface>
+      </joint>
+      <actuator name="${arm_id}_motor6">
+	    <hardwareInterface>PositionJointInterface</hardwareInterface>
+	    <mechanicalReduction>1</mechanicalReduction>
+      </actuator>
+    </transmission>
     <link name="${arm_id}_link7">
       <visual>
@@ -209,4 +275,15 @@
       <limit effort="12" lower="-2.8973" upper="2.8973" velocity="2.6100"/>
     </joint>
+    <transmission name="${arm_id}_transmission7">
+      <robotNamespace>/</robotNamespace>
+      <type>transmission_interface/SimpleTransmission</type>
+      <joint name="${arm_id}_joint7">
+	    <hardwareInterface>PositionJointInterface</hardwareInterface>
+      </joint>
+      <actuator name="${arm_id}_motor7">
+	    <hardwareInterface>PositionJointInterface</hardwareInterface>
+	    <mechanicalReduction>1</mechanicalReduction>
+      </actuator>
+    </transmission>
     <link name="${arm_id}_link8"/>
     <joint name="${arm_id}_joint8" type="fixed">

Commit message: Switch to reconverted .dae files.

File: franka_description/robots/panda_arm.xacro (robot description, xacro)
@@ -12,5 +12,5 @@
       <visual>
         <geometry>
-          <mesh filename="package://${description_pkg}/meshes/visual/link0.dae"/>
+          <mesh filename="package://${description_pkg}/meshes/visual/link0.dae.dae"/>
         </geometry>
       </visual>
@@ -38,5 +38,5 @@
       <visual>
         <geometry>
-          <mesh filename="package://${description_pkg}/meshes/visual/link1.dae"/>
+          <mesh filename="package://${description_pkg}/meshes/visual/link1.dae.dae"/>
         </geometry>
       </visual>
@@ -84,5 +84,5 @@
       <visual>
         <geometry>
-          <mesh filename="package://${description_pkg}/meshes/visual/link2.dae"/>
+          <mesh filename="package://${description_pkg}/meshes/visual/link2.dae.dae"/>
         </geometry>
       </visual>
@@ -130,5 +130,5 @@
       <visual>
         <geometry>
-          <mesh filename="package://${description_pkg}/meshes/visual/link3.dae"/>
+          <mesh filename="package://${description_pkg}/meshes/visual/link3.dae.dae"/>
         </geometry>
       </visual>
@@ -176,5 +176,5 @@
       <visual>
         <geometry>
-          <mesh filename="package://${description_pkg}/meshes/visual/link4.dae"/>
+          <mesh filename="package://${description_pkg}/meshes/visual/link4.dae.dae"/>
         </geometry>
       </visual>
@@ -222,5 +222,5 @@
       <visual>
         <geometry>
-          <mesh filename="package://${description_pkg}/meshes/visual/link5.dae"/>
+          <mesh filename="package://${description_pkg}/meshes/visual/link5.dae.dae"/>
         </geometry>
       </visual>
@@ -268,5 +268,5 @@
       <visual>
         <geometry>
-          <mesh filename="package://${description_pkg}/meshes/visual/link6.dae"/>
+          <mesh filename="package://${description_pkg}/meshes/visual/link6.dae.dae"/>
         </geometry>
       </visual>
@@ -314,5 +314,5 @@
       <visual>
         <geometry>
-          <mesh filename="package://${description_pkg}/meshes/visual/link7.dae"/>
+          <mesh filename="package://${description_pkg}/meshes/visual/link7.dae.dae"/>
         </geometry>
       </visual>
