Commit message: Add moveit tutorial script.

File: franka_description/robots/panda_arm_hand.urdf.xacro (robot description, xacro)
@@ -3,6 +3,6 @@
   <xacro:include filename="$(find franka_description)/robots/panda_arm.xacro"/>
   <xacro:include filename="$(find franka_description)/robots/hand.xacro"/>
-  <link name="world"/>
-  <xacro:panda_arm connected_to="world"/>
+  <!--link name="world"/-->
+  <xacro:panda_arm connected_to=""/>
   <xacro:hand ns="panda" rpy="0 0 ${-pi/4}" connected_to="panda_link8"/>
   <gazebo>

Commit message: Restore functionality of load_gripper arg in launch file.

File: franka_description/robots/panda_arm_hand.urdf.xacro (robot description, xacro)
@@ -3,6 +3,6 @@
   <xacro:include filename="$(find franka_description)/robots/panda_arm.xacro"/>
   <xacro:include filename="$(find franka_description)/robots/hand.xacro"/>
-  <!--link name="world"/-->
-  <xacro:panda_arm connected_to=""/>
+  <link name="world"/>
+  <xacro:panda_arm connected_to="world"/>
   <xacro:hand ns="panda" rpy="0 0 ${-pi/4}" connected_to="panda_link8"/>
   <gazebo>
