Commit message: Add possibility of velocity control with both the real and the simulated robot.

File: franka_description/robots/panda_arm.urdf.xacro (robot description, xacro)
@@ -1,7 +1,8 @@
 <?xml version='1.0' encoding='utf-8'?>
 <robot xmlns:xacro="http://www.ros.org/wiki/xacro" name="panda">
+  <xacro:arg name="hw_interface" default="PositionJointInterface"/>
   <xacro:include filename="$(find franka_description)/robots/panda_arm.xacro" />
   <link name="world"/>
-  <xacro:panda_arm connected_to="world"/>
+  <xacro:panda_arm connected_to="world" hw_interface="$(arg hw_interface)"/>
   <gazebo>
     <plugin name="gazebo_ros_control" filename="libgazebo_ros_control.so">

File: franka_description/robots/panda_arm.xacro (robot description, xacro)
@@ -1,5 +1,5 @@
 <?xml version='1.0' encoding='utf-8'?>
 <robot xmlns:xacro="http://www.ros.org/wiki/xacro" name="panda">
-  <xacro:macro name="panda_arm" params="arm_id:='panda' description_pkg:='franka_description' connected_to:='' xyz:='0 0 0' rpy:='0 0 0'">
+  <xacro:macro name="panda_arm" params="arm_id:='panda' description_pkg:='franka_description' connected_to:='' xyz:='0 0 0' rpy:='0 0 0' hw_interface:='PositionJointInterface'">
     <xacro:unless value="${not connected_to}">
       <joint name="${arm_id}_joint_${connected_to}" type="fixed">
@@ -74,8 +74,8 @@
       <type>transmission_interface/SimpleTransmission</type>
       <joint name="${arm_id}_joint1">
-	    <hardwareInterface>hardware_interface/PositionJointInterface</hardwareInterface>
+	    <hardwareInterface>hardware_interface/${hw_interface}</hardwareInterface>
       </joint>
       <actuator name="${arm_id}_motor1">
-	    <hardwareInterface>hardware_interface/PositionJointInterface</hardwareInterface>
+	    <hardwareInterface>hardware_interface/${hw_interface}</hardwareInterface>
 	    <mechanicalReduction>1</mechanicalReduction>
       </actuator>
@@ -120,8 +120,8 @@
       <type>transmission_interface/SimpleTransmission</type>
       <joint name="${arm_id}_joint2">
-	    <hardwareInterface>hardware_interface/PositionJointInterface</hardwareInterface>
+	    <hardwareInterface>hardware_interface/${hw_interface}</hardwareInterface>
       </joint>
       <actuator name="${arm_id}_motor2">
-	    <hardwareInterface>hardware_interface/PositionJointInterface</hardwareInterface>
+	    <hardwareInterface>hardware_interface/${hw_interface}</hardwareInterface>
 	    <mechanicalReduction>1</mechanicalReduction>
       </actuator>
@@ -166,8 +166,8 @@
       <type>transmission_interface/SimpleTransmission</type>
       <joint name="${arm_id}_joint3">
-	    <hardwareInterface>hardware_interface/PositionJointInterface</hardwareInterface>
+	    <hardwareInterface>hardware_interface/${hw_interface}</hardwareInterface>
       </joint>
       <actuator name="${arm_id}_motor3">
-	    <hardwareInterface>hardware_interface/PositionJointInterface</hardwareInterface>
+	    <hardwareInterface>hardware_interface/${hw_interface}</hardwareInterface>
 	    <mechanicalReduction>1</mechanicalReduction>
       </actuator>
@@ -212,8 +212,8 @@
       <type>transmission_interface/SimpleTransmission</type>
       <joint name="${arm_id}_joint4">
-	    <hardwareInterface>hardware_interface/PositionJointInterface</hardwareInterface>
+	    <hardwareInterface>hardware_interface/${hw_interface}</hardwareInterface>
       </joint>
       <actuator name="${arm_id}_motor4">
-	    <hardwareInterface>hardware_interface/PositionJointInterface</hardwareInterface>
+	    <hardwareInterface>hardware_interface/${hw_interface}</hardwareInterface>
 	    <mechanicalReduction>1</mechanicalReduction>
       </actuator>
@@ -258,8 +258,8 @@
       <type>transmission_interface/SimpleTransmission</type>
       <joint name="${arm_id}_joint5">
-	    <hardwareInterface>hardware_interface/PositionJointInterface</hardwareInterface>
+	    <hardwareInterface>hardware_interface/${hw_interface}</hardwareInterface>
       </joint>
       <actuator name="${arm_id}_motor5">
-	    <hardwareInterface>hardware_interface/PositionJointInterface</hardwareInterface>
+	    <hardwareInterface>hardware_interface/${hw_interface}</hardwareInterface>
 	    <mechanicalReduction>1</mechanicalReduction>
       </actuator>
@@ -304,8 +304,8 @@
       <type>transmission_interface/SimpleTransmission</type>
       <joint name="${arm_id}_joint6">
-	    <hardwareInterface>hardware_interface/PositionJointInterface</hardwareInterface>
+	    <hardwareInterface>hardware_interface/${hw_interface}</hardwareInterface>
       </joint>
       <actuator name="${arm_id}_motor6">
-	    <hardwareInterface>hardware_interface/PositionJointInterface</hardwareInterface>
+	    <hardwareInterface>hardware_interface/${hw_interface}</hardwareInterface>
 	    <mechanicalReduction>1</mechanicalReduction>
       </actuator>
@@ -350,8 +350,8 @@
       <type>transmission_interface/SimpleTransmission</type>
       <joint name="${arm_id}_joint7">
-	    <hardwareInterface>hardware_interface/PositionJointInterface</hardwareInterface>
+	    <hardwareInterface>hardware_interface/${hw_interface}</hardwareInterface>
       </joint>
       <actuator name="${arm_id}_motor7">
-	    <hardwareInterface>hardware_interface/PositionJointInterface</hardwareInterface>
+	    <hardwareInterface>hardware_interface/${hw_interface}</hardwareInterface>
 	    <mechanicalReduction>1</mechanicalReduction>
       </actuator>

File: franka_description/robots/panda_arm_hand.urdf.xacro (robot description, xacro)
@@ -1,8 +1,9 @@
 <?xml version="1.0" encoding="utf-8"?>
 <robot xmlns:xacro="http://www.ros.org/wiki/xacro" name="panda">
+  <xacro:arg name="hw_interface" default="PositionJointInterface"/>
   <xacro:include filename="$(find franka_description)/robots/panda_arm.xacro"/>
   <xacro:include filename="$(find franka_description)/robots/hand.xacro"/>
   <link name="world"/>
-  <xacro:panda_arm connected_to="world"/>
+  <xacro:panda_arm connected_to="world" hw_interface="$(arg hw_interface)"/>
   <xacro:hand ns="panda" rpy="0 0 ${-pi/4}" connected_to="panda_link8"/>
   <gazebo>
