Commit message: Add transmissions for fingers.

File: franka_description/robots/hand.xacro (robot description, xacro)
@@ -72,4 +72,15 @@
       <limit effort="20" lower="0.0" upper="0.04" velocity="0.2"/>
     </joint>
+    <transmission name="${ns}_finger_transmission1">
+      <robotNamespace>/</robotNamespace>
+      <type>transmission_interface/SimpleTransmission</type>
+      <joint name="${ns}_finger_joint1">
+	    <hardwareInterface>PositionJointInterface</hardwareInterface>
+      </joint>
+      <actuator name="${ns}_finger_motor1">
+	    <hardwareInterface>PositionJointInterface</hardwareInterface>
+	    <mechanicalReduction>1</mechanicalReduction>
+      </actuator>
+    </transmission>
     <joint name="${ns}_finger_joint2" type="prismatic">
       <parent link="${ns}_hand"/>
@@ -80,4 +91,15 @@
       <mimic joint="${ns}_finger_joint1" />
     </joint>
+    <transmission name="${ns}_finger_transmission2">
+      <robotNamespace>/</robotNamespace>
+      <type>transmission_interface/SimpleTransmission</type>
+      <joint name="${ns}_finger_joint2">
+	    <hardwareInterface>PositionJointInterface</hardwareInterface>
+      </joint>
+      <actuator name="${ns}_finger_motor2">
+	    <hardwareInterface>PositionJointInterface</hardwareInterface>
+	    <mechanicalReduction>1</mechanicalReduction>
+      </actuator>
+    </transmission>
   </xacro:macro>
 </robot>

Commit message: Add gripper control.

File: franka_description/robots/hand.xacro (robot description, xacro)
@@ -12,5 +12,5 @@
       <visual>
         <geometry>
-          <mesh filename="package://franka_description/meshes/visual/hand.dae"/>
+          <mesh filename="package://franka_description/meshes/visual/hand.dae.dae"/>
         </geometry>
       </visual>
@@ -30,5 +30,5 @@
       <visual>
         <geometry>
-          <mesh filename="package://franka_description/meshes/visual/finger.dae"/>
+          <mesh filename="package://franka_description/meshes/visual/finger.dae.dae"/>
         </geometry>
       </visual>
@@ -49,5 +49,5 @@
         <origin xyz="0 0 0" rpy="0 0 ${pi}"/>
         <geometry>
-          <mesh filename="package://franka_description/meshes/visual/finger.dae"/>
+          <mesh filename="package://franka_description/meshes/visual/finger.dae.dae"/>
         </geometry>
       </visual>
@@ -76,9 +76,9 @@
       <type>transmission_interface/SimpleTransmission</type>
       <joint name="${ns}_finger_joint1">
-	    <hardwareInterface>PositionJointInterface</hardwareInterface>
+	        <hardwareInterface>hardware_interface/PositionJointInterface</hardwareInterface>
       </joint>
       <actuator name="${ns}_finger_motor1">
-	    <hardwareInterface>PositionJointInterface</hardwareInterface>
-	    <mechanicalReduction>1</mechanicalReduction>
+	       <hardwareInterface>hardware_interface/PositionJointInterface</hardwareInterface>
+	        <mechanicalReduction>1</mechanicalReduction>
       </actuator>
     </transmission>
@@ -95,8 +95,8 @@
       <type>transmission_interface/SimpleTransmission</type>
       <joint name="${ns}_finger_joint2">
-	    <hardwareInterface>PositionJointInterface</hardwareInterface>
+	       <hardwareInterface>hardware_interface/PositionJointInterface</hardwareInterface>
       </joint>
       <actuator name="${ns}_finger_motor2">
-	    <hardwareInterface>PositionJointInterface</hardwareInterface>
+	    <hardwareInterface>hardware_interface/PositionJointInterface</hardwareInterface>
 	    <mechanicalReduction>1</mechanicalReduction>
       </actuator>

File: franka_description/robots/panda_arm_hand.urdf.xacro (robot description, xacro)
@@ -3,5 +3,6 @@
   <xacro:include filename="$(find franka_description)/robots/panda_arm.xacro"/>
   <xacro:include filename="$(find franka_description)/robots/hand.xacro"/>
-  <xacro:panda_arm />
+  <link name="world"/>
+  <xacro:panda_arm connected_to="world"/>
   <xacro:hand ns="panda" rpy="0 0 ${-pi/4}" connected_to="panda_link8"/>
   <gazebo>

Commit message: Add friction parameters and activate gripperFix plugin for gripper.

File: franka_description/robots/hand.xacro (robot description, xacro)
@@ -37,4 +37,5 @@
           <mesh filename="package://franka_description/meshes/collision/finger.stl"/>
         </geometry>
+        <contact_coefficient mu="10.0"  k_p="100"  k_d="1" />
       </collision>
       <inertial>
@@ -57,4 +58,5 @@
           <mesh filename="package://franka_description/meshes/collision/finger.stl"/>
         </geometry>
+        <contact_coefficient mu="10.0"  k_p="100"  k_d="1" />
       </collision>
       <inertial>
@@ -71,4 +73,5 @@
       <axis xyz="0 1 0"/>
       <limit effort="20" lower="0.0" upper="0.04" velocity="0.2"/>
+      <dynamics damping="1" friction="0"/>
     </joint>
     <transmission name="${ns}_finger_transmission1">
@@ -89,4 +92,5 @@
       <axis xyz="0 -1 0"/>
       <limit effort="20" lower="0.0" upper="0.04" velocity="0.2"/>
+      <dynamics damping="1" friction="0"/>
       <mimic joint="${ns}_finger_joint1" />
     </joint>
@@ -102,4 +106,50 @@
       </actuator>
     </transmission>
+    <link name="${ns}_tcp"/>
+    <joint name="${ns}_hand_tcp_joint" type="fixed">
+      <parent link="${ns}_hand"/>
+      <child link="${ns}_tcp"/>
+      <origin xyz="0 0 0.1025" rpy="0 0 0"/>
+    </joint>
+    <gazebo reference="${ns}_leftfinger">
+        <kp>1000000.0</kp>
+        <kd>1.0</kd>
+        <mu1>1.0</mu1>
+        <mu2>1.0</mu2>
+        <minDepth>0.001</minDepth>
+    </gazebo>
+    <gazebo reference="${ns}_rightfinger">
+        <kp>1000000.0</kp>
+        <kd>1.0</kd>
+        <mu1>1.0</mu1>
+        <mu2>1.0</mu2>
+        <minDepth>0.001</minDepth>
+    </gazebo>
+    <gazebo reference="${ns}_finger_joint1">
+        <implicitSpringDamper>1</implicitSpringDamper>
+    </gazebo>
+    <gazebo reference="${ns}_finger_joint2">
+        <implicitSpringDamper>1</implicitSpringDamper>
+    </gazebo>
+    <!-- Load gripper plugin. This plugin fixes an object which is grasped to the
+         robot hand to avoid problems with physics engines and to help the object
+         stay in the robot hand without slipping out -->
+    <gazebo>
+       <plugin name="gazebo_grasp_fix" filename="libgazebo_grasp_fix.so">
+            <arm>
+               <arm_name>gripper</arm_name>
+               <palm_link>${ns}_link7</palm_link>
+               <gripper_link>${ns}_leftfinger</gripper_link>
+               <gripper_link>${ns}_rightfinger</gripper_link>
+            </arm>
+           <forces_angle_tolerance>150</forces_angle_tolerance>
+           <update_rate>10</update_rate>
+           <grip_count_threshold>3</grip_count_threshold>
+           <max_grip_count>4</max_grip_count>
+           <release_tolerance>0.001</release_tolerance>
+           <disable_collisions_on_attach>false</disable_collisions_on_attach>
+           <contact_topic>__default_topic__</contact_topic>
+        </plugin>
+    </gazebo>
   </xacro:macro>
 </robot>

Commit message: Tweak inertia values a little.

File: franka_description/robots/hand.xacro (robot description, xacro)
@@ -19,9 +19,10 @@
           <mesh filename="package://franka_description/meshes/collision/hand.stl"/>
         </geometry>
+        <contact_coefficient mu="0.8"  k_p="1"  k_d="1" />
       </collision>
       <inertial>
         <!-- ATTENTION! Needs to be defined correctly! -->
-        <origin xyz="0 0 0.02" rpy="0 0 0"/>
-        <mass value="0.3"/>
+        <origin xyz="0 0 0.025" rpy="0 0 0"/>
+        <mass value="1.0"/>
         <inertia ixx="0.001"  ixy="0"  ixz="0" iyy="0.001" iyz="0" izz="0.001" />
       </inertial>
@@ -37,5 +38,5 @@
           <mesh filename="package://franka_description/meshes/collision/finger.stl"/>
         </geometry>
-        <contact_coefficient mu="10.0"  k_p="100"  k_d="1" />
+        <contact_coefficient mu="0.8"  k_p="100"  k_d="1" />
       </collision>
       <inertial>
@@ -58,5 +59,5 @@
           <mesh filename="package://franka_description/meshes/collision/finger.stl"/>
         </geometry>
-        <contact_coefficient mu="10.0"  k_p="100"  k_d="1" />
+        <contact_coefficient mu="0.8"  k_p="100"  k_d="1" />
       </collision>
       <inertial>
@@ -113,6 +114,6 @@
         <kp>1000000.0</kp>
         <kd>1.0</kd>
-        <mu1>1.0</mu1>
-        <mu2>1.0</mu2>
+        <mu1>0.3</mu1>
+        <mu2>0.3</mu2>
         <minDepth>0.001</minDepth>
     </gazebo>
@@ -120,6 +121,6 @@
         <kp>1000000.0</kp>
         <kd>1.0</kd>
-        <mu1>1.0</mu1>
-        <mu2>1.0</mu2>
+        <mu1>0.3</mu1>
+        <mu2>0.3</mu2>
         <minDepth>0.001</minDepth>
     </gazebo>

File: franka_description/robots/panda_arm.xacro (robot description, xacro)
@@ -28,5 +28,4 @@
     </link>
     <gazebo reference="${arm_id}_link0">
-      <kp>1000000.0</kp>
       <kd>1.0</kd>
       <mu1>0.8</mu1>
@@ -49,10 +48,9 @@
         <!-- ATTENTION! Copied from another robot! Needs to be defined correctly! -->
         <mass value="2.0" />
-        <origin rpy="0 0 0" xyz="0 0 0.130" />
+        <origin rpy="0 0 0" xyz="0 0 -0.130" />
         <inertia ixx="0.0136666666667" ixy="0" ixz="0" iyy="0.0118666666667" iyz="0" izz="0.003" />
       </inertial>
     </link>
     <gazebo reference="${arm_id}_link1">
-      <kp>1000000.0</kp>
       <kd>1.0</kd>
       <mu1>0.8</mu1>
@@ -94,10 +92,9 @@
         <!-- ATTENTION! Copied from another robot! Needs to be defined correctly! -->
         <mass value="2.0" />
-        <origin rpy="0 0 0" xyz="0 -0.06 0.07" />
+        <origin rpy="0 0 0" xyz="0 -0.05 0.04" />
         <inertia ixx="0.0136666666667" ixy="0" ixz="0" iyy="0.0118666666667" iyz="0" izz="0.003" />
       </inertial>
     </link>
     <gazebo reference="${arm_id}_link2">
-      <kp>1000000.0</kp>
       <kd>1.0</kd>
       <mu1>0.8</mu1>
@@ -139,10 +136,9 @@
         <!-- ATTENTION! Copied from another robot! Needs to be defined correctly! -->
         <mass value="2.0" />
-        <origin rpy="0 0 0" xyz="0 -0.06 0.130" />
-        <inertia ixx="0.0136666666667" ixy="0" ixz="0" iyy="0.0118666666667" iyz="0" izz="0.003" />
+        <origin rpy="0 0 0" xyz="0 0.0 0.0" />
+        <inertia ixx="0.011" ixy="0" ixz="0" iyy="0.0118666666667" iyz="0" izz="0.003" />
       </inertial>
     </link>
     <gazebo reference="${arm_id}_link3">
-      <kp>1000000.0</kp>
       <kd>1.0</kd>
       <mu1>0.8</mu1>
@@ -184,10 +180,9 @@
         <!-- ATTENTION! Copied from another robot! Needs to be defined correctly! -->
         <mass value="2.0" />
-        <origin rpy="0 0 0" xyz="0 0.06 0.07" />
-        <inertia ixx="0.0136666666667" ixy="0" ixz="0" iyy="0.0118666666667" iyz="0" izz="0.003" />
+        <origin rpy="0 0 0" xyz="-0.04 0.06 0.0" />
+        <inertia ixx="0.01" ixy="0" ixz="0" iyy="0.011" iyz="0" izz="0.0129" />
       </inertial>
     </link>
     <gazebo reference="${arm_id}_link4">
-      <kp>1000000.0</kp>
       <kd>1.0</kd>
       <mu1>0.8</mu1>
@@ -229,10 +224,9 @@
         <!-- ATTENTION! Copied from another robot! Needs to be defined correctly! -->
         <mass value="2.0" />
-        <origin rpy="0 0 0" xyz="0 0 0.124" />
+        <origin rpy="0 0 0" xyz="0 0.03 -0.123" />
         <inertia ixx="0.0126506666667" ixy="0" ixz="0" iyy="0.0108506666667" iyz="0" izz="0.003" />
       </inertial>
     </link>
     <gazebo reference="${arm_id}_link5">
-      <kp>1000000.0</kp>
       <kd>1.0</kd>
       <mu1>0.8</mu1>
@@ -273,11 +267,10 @@
       <inertial>
         <!-- ATTENTION! Copied from another robot! Needs to be defined correctly! -->
-        <mass value="1.0" />
-        <origin rpy="0 0 0" xyz="0 0 0.0" />
-        <inertia ixx="0.00260416666667" ixy="0" ixz="0" iyy="0.00260416666667" iyz="0" izz="0.00260416666667" />
+        <mass value="1.5" />
+        <origin rpy="0 0 0" xyz="0.05 0 0.0" />
+        <inertia ixx="0.002" ixy="0" ixz="0" iyy="0.00260416666667" iyz="0" izz="0.00260416666667" />
       </inertial>
     </link>
     <gazebo reference="${arm_id}_link6">
-      <kp>1000000.0</kp>
       <kd>1.0</kd>
       <mu1>0.8</mu1>
@@ -318,5 +311,5 @@
       <inertial>
         <!-- ATTENTION! Copied from another robot! Needs to be defined correctly! -->
-        <mass value="0.2" />
+        <mass value="0.8" />
         <origin xyz="0 0 0" />
         <inertia ixx="6.66666666667e-05" ixy="0" ixz="0" iyy="6.66666666667e-05" iyz="0" izz="0.00012" />
@@ -324,5 +317,4 @@
     </link>
     <gazebo reference="${arm_id}_link7">
-      <kp>1000000.0</kp>
       <kd>1.0</kd>
       <mu1>0.8</mu1>
